File: pcb_macropad/pcb_macropad.kicad_sch (KiCad schematic)
At the start: 23 parts, among them J1 OLED_128x32, SW1 RotaryEncoder_Switch, U1 Arduino_Pro_Micro

Commit message: Updates
Parts:
- removed D10: LED, LED_THT:LED_D5.0mm, symbol Device:LED
- removed J1: OLED_128x32, ScottoKeebs_Components:OLED_128x32, symbol ScottoKeebs:OLED_128x32
- removed R1: R330, Resistor_THT:R_Axial_DIN0207_L6.3mm_D2.5mm_P7.62mm_Horizontal, symbol Device:R
- added J1: OLED_128x64, SSD1306:128x64OLED, symbol ScottoKeebs:OLED_128x64
- SW1: footprint Rotary_Encoder:RotaryEncoder_Alps_EC12E-Switch_Vertical_H20mm -> Rotary_Encoder:RotaryEncoder_Alps_EC11E-Switch_Vertical_H20mm
Connections:
- net EncoderA: now also U1.8 (5/PC6); no longer U1.7 (4/PD4)
- net EncoderB: now also U1.9 (6/PD7); no longer U1.8 (5/PC6)
- net EncoderSW: now also U1.10 (7/PE6); no longer U1.9 (6/PD7)
- net GND: now also J1.1 (GND)
- net SCL: now also J1.3 (SCL)
- net SDA: now also J1.4 (SDA)
- net Row 3: now reaches U1.16 (15/PB1)
- net Row 3: now also D7.1 (K), D8.1 (K), D9.1 (K)
- net Row 2: now reaches U1.17 (A0/PF7)
- net Row 2: now also D4.1 (K), D5.1 (K), D6.1 (K)
- net Row 1: now reaches U1.18 (A1/PF6)
- net Row 1: now also D1.1 (K), D2.1 (K), D3.1 (K)
- net +5V renamed VCC
- net VCC: now also J1.2 (VCC)
- net Col1 renamed Column 1
- net Column 1: now also U1.15 (14/PB3); no longer U1.10 (7/PE6)
- net Col2 renamed Column 2
- net Column 2: now also U1.14 (16/PB2); no longer U1.11 (8/PB4)
- net Col3 renamed Column 3
- net Column 3: now also U1.13 (10/PB6); no longer U1.12 (9/PB5)
- removed net Row1: D1.1 (K), D2.1 (K), D3.1 (K), U1.15 (14/PB3)
- removed net Row2: D4.1 (K), D5.1 (K), D6.1 (K), U1.14 (16/PB2)
- removed net Row3: D7.1 (K), D8.1 (K), D9.1 (K), U1.13 (10/PB6)
